File: eagle/euro buffered mult/buffered mult rt1_postpwer.sch (EAGLE design)
At the start: 88 parts, among them IC1 7805, Q1 2.5A/30V, U1 TL074_SMD, U2 TL074_SMD

Commit message: add euro buffer
Parts:
- removed C12, C17, C22: 10uf, resistor:CPOL-US153CLV-0505
- removed C13, C14, C18, C19: 0.1uf, resistor:C-USC0603
- removed C15, C16, C20, C21: 0.01uf, resistor:C-USC0603
- removed C26: 1800pf, resistor:C-USC0603
- removed C27: 2700pf, resistor:C-USC0603
- removed C28: 5600pf, resistor:C-USC0603
- removed C29, C30: 22uf, resistor:CPOL-US153CLV-0605
- removed C31: 1200pf, resistor:C-USC0603
- removed D1: RED, SparkFun-LED:LED-RED0603
- removed D4: 1N4004, diode:1N4004
- removed IC1: 7805, v-reg:78XXS
- removed JP1: OUTPUT JACK 2, SparkFun-Connectors:AUDIO-JACK4-.25-HORIZ-TRS
- removed JP14: PTH-LED, SparkFun-Connectors:M02PTH3
- removed JP17: OUTPUT JACK, SparkFun-Connectors:AUDIO-JACK4-.25-HORIZ-TRS
- removed JP2: INPUT JACK, SparkFun-Connectors:AUDIO-JACK4-.25-HORIZ-TRS
- removed JP3: 9VBattery, SparkFun-Connectors:M02PTH3
- removed JP4: POWER_JACK_TIP_NEGATIVE, Testing:POWER_JACK_TIP_NEGATIVE
- removed JP6, JP9: 1x3, SparkFun-Connectors:M031X03_NO_SILK
- removed Q1: 2.5A/30V, SparkFun-DiscreteSemi:MOSFET-PCHANNELDMG2307L
- removed S1: SWITCH-3PDT, SparkFun-Electromechanical:SWITCH-3PDT
- removed SJ1: disable LED, SparkFun-Passives:JUMPER-PAD-2-NC_BY_PASTEFULL-BOX-SILK
- removed TP1: Raw In, SparkFun-Connectors:M01PTH_NO_SILK_YES_STOP
- removed TP2: Raw Out, SparkFun-Connectors:M01PTH_NO_SILK_YES_STOP
- removed TP3: Out Ring, SparkFun-Connectors:M01PTH_NO_SILK_YES_STOP
- removed TP4: In Ring, SparkFun-Connectors:M01PTH_NO_SILK_YES_STOP
- removed TP5: FX Input, SparkFun-Connectors:M01PTH_NO_SILK_YES_STOP
- removed TP6: FX Output, SparkFun-Connectors:M01PTH_NO_SILK_YES_STOP
- removed U$1: CS42448, akm:CS42448
- removed U$2: TEENSY_3.5/3.6, Teensy356:TEENSY_3.5/3.6
- removed U$3: CAT811, sot143:CAT811
- removed VR1: 1M, MusicThingModular:9MM_SNAP-IN_POT_
- added IN1, IN2, OUT1-1, OUT1-2, OUT1-3, OUT2-1, OUT2-2, OUT2-3: THONKICONNNEW, MusicThingModular:THONKICONNNEW
- added TR1, TR2, TR3, TR4, TR5, TR6: 2k, MusicThingModular:BOURNS_3362P_TRIMMERP
- C1: value C in -> 6pf; device Testing:DUAL_FOOTPRINT_CAP -> resistor:C-USC0603
- C11, C7: value 22uf -> 0.1uf; device resistor:CPOL-US153CLV-0605 -> resistor:C-USC0603
- C2: value C out -> 10pf; device Testing:DUAL_FOOTPRINT_CAP -> resistor:C-USC0603
- C23: value 4.7uf 0805 -> 10pf; device resistor:C-USC0805 -> resistor:C-USC0603
- C24: value 470pf -> 10pf
- C25: value 2700pf -> 0.1uf
- C3, C5: value 0.1uf -> 10pf
- C4: value o.1uf -> 6pf
- C6: value 100uf -> 10pf; device resistor:CPOL-US153CLV-0810 -> resistor:C-USC0603
- C8: value 4.7uf -> 0.1uf; device resistor:CPOL-US153CLV-0505 -> resistor:C-USC0603
- R1: value 1M -> 100k; device SparkFun-Resistors:1MOHM-1/10W-1%(0603) -> resistor:R-US_R0603
- R10, R13, R6: value 100k -> 301R
- R11: value 634 -> 49.9k
- R12: value 150R -> 49.9k
- R14: value 100k -> 13.3k
- R16: value 20k -> 107k
- R17: value 1k -> 49.9k
- R18: value 1k -> 13.3k
- R19: value 2.94k -> 49.9k
- R2: value 1M -> 107k; device SparkFun-Resistors:1MOHM-1/10W-1%(0603) -> resistor:R-US_R0603
- R20: value 887R -> 301R
- R21: value 5.49k -> 49.9k
- R22: value 47k -> 49.9k
- R23: value 1M -> 13.3k
- R24: value 1.65k -> 301R
- R25: value 4.75k -> 49.9k
- R26: value 1.87k -> 49.9k
- R27: value 562R -> 301R
- R28: value 47.5k -> 13.3k
- R3: value 1M -> 13.3k; device SparkFun-Resistors:1MOHM-1/10W-1%(0603) -> resistor:R-US_R0603
- R4: value BRT -> 49.9k; device SparkFun-Resistors:RESISTORAXIAL-0.3 -> resistor:R-US_R0603
- R5: value 1K -> 49.9k; device SparkFun-Resistors:1KOHM-1/10W-1%(0603) -> resistor:R-US_R0603
- R7: value 91 -> 49.9k
- R8: value 100k -> 49.9k
- R9: value 27k -> 13.3k
Connections:
- removed net BCLK: U$1.ADC_SCLK, U$1.DAC_SCLK, U$2.9/CS
- removed net FX_IN: C1.-, R2.2, S1A.P
- removed net FX_OUT: C2.-, R3.2, S1B.S
- removed net LEDA: JP14.1, R4.2
- removed net LRCLK: U$1.ADC_LRCK, U$1.DAC_LRCK, U$2.23/A9
- removed net MCLK: U$1.MCLK, U$2.11/MOSI
- removed net N$22: R22.2
- removed net N$35: R4.1, S1C.S, SJ1.1
- removed net N$45: JP3.1, JP4.SLEEVEBREAK
- removed net N$55: JP2.RING, JP3.2, JP4.TIP, TP4.1
- removed net N$65: R5.1, SJ1.2
- removed net N$66: JP17.RING, TP3.1
- removed net N$67: C1.+, TP5.1
- removed net N$68: C2.+, TP6.1
- removed net N$70: JP2.TIP, S1A.S, S1B.O, TP1.1
- removed net N$71: JP17.TIP, S1B.P, TP2.1
- removed net N$75: Q1.G, R1.2
- removed net PWR33V: C13.1, C14.1, C15.1, C16.1, C17.+, R13.1, U$1.VD, U$1.VD1, U$1.VLC, U$1.VLS, U$2.3V3
- removed net PWR5V: C18.1, C19.1, C20.1, C21.1, C22.+, D4.C, R8.2, U$1.VA, U$1.VA1, U$2.VIN
- removed net RESET: U$1.RST
- removed net RX: U$1.ADC_SDOUT1, U$2.13/SCK
- removed net SCL: U$1.SCL/CCLK, U$2.19/A5/SCL
- removed net SDA: U$1.SDA/CDOUT, U$2.18/A4/SDA
- removed net TOAIN1: C25.1, R11.2, R7.2
- removed net TX: U$1.DAC_SDIN1, U$2.22/A8
- removed net VAUX: JP6.3, JP9.3
- removed net VBATT: JP4.SLEEVE, Q1.D
- removed net VCC: JP6.2, JP9.2, Q1.S, S1C.P
- removed net VQ: C5.1, C8.+, U$1.VQ
- new net N$11: C3.2, R17.1, R19.1, U2B.-IN
- new net N$24: C5.1, R24.1, U2C.OUT
- new net N$27: R28.1, TR6.1
- new net N$29: C6.2, R25.1, R26.1, U2D.-IN
- new net N$3: C1.2, R1.1, R2.1, U1A.-IN
- new net N$30: C6.1, R27.1, U2D.OUT
- new net N$41: R14.1, TR3.1
- new net N$42: R12.2, TR3.2, TR3.2-2
- new net N$43: C23.2, R11.1, R12.1, U1D.-IN
- new net TO-IN2: C23.1, IN2.SWITCH, OUT1-3.TIP, R11.2, R13.1, R13.2, U1D.OUT
- new net TO-IN3: IN2.TIP, R15.2
- net GND: now also C11.1, C7.1, C8.2, IN1.SLEEVE, IN2.SLEEVE, OUT1-1.SLEEVE, OUT1-2.SLEEVE, OUT1-3.SLEEVE, OUT2-1.SLEEVE, OUT2-2.SLEEVE, OUT2-3.SLEEVE, R14.2, R18.2, R23.2, R3.2, R9.2, U1A.+IN, U1B.+IN, U1D.+IN, U2A.+IN, U2B.+IN, U2C.+IN, U2D.+IN; no longer C11.-, C12.-, C13.2, C14.2, C15.2, C16.2, C17.-, C18.2, C19.2, C20.2, C21.2, C22.-, C26.1, C28.1, C29.-, C31.2, D1.C, IC1.GND, JP14.2, JP17.EARTH, JP2.EARTH, JP6.1, JP9.1, R1.1, R10.1, R12.1, R16.2, R2.1, R3.1, R6.1, S1A.O, U$1.AUX_SCLK, U$1.AUX_SDIN, U$1.CDIN, U$1.DAC_SDIN2, U$1.DAC_SDIN3, U$1.DAC_SDIN4
- net N$1: now also IN1.TIP, R1.2; no longer R12.2, R13.2, U$1.CS
- net N$10: now also C24.2, R4.1, R5.1, U1B.-IN; no longer C23.1, R10.2, R8.1, U1A.+IN
- net N$12: now also C24.1, R6.1, U1B.OUT; no longer R15.2, R16.1, U1B.+IN
- net N$13: now also OUT1-1.TIP, R5.2, R6.2; no longer R18.2, R9.1, U1B.OUT
- net N$14: now also C3.1, R20.1, U2B.OUT; no longer R14.2, R9.2, U1B.-IN
- net N$15: now also R9.1, TR2.1; no longer R14.1
- net N$16: now also OUT2-1.TIP, R17.2, R20.2; no longer C30.-, R27.2
- net N$17: now also R23.1, TR5.1; no longer R27.1, R28.1
- net N$18: now also R22.2, TR5.2, TR5.2-2; no longer C31.1, R20.1, U2A.-IN
- net N$19: now also R8.2, TR2.2, TR2.2-2; no longer R23.2, U1C.-IN, VR1.E
- net N$2: now also C4.1, R16.2, TR4.3, TR5.3, TR6.3, U2A.OUT; no longer C3.2, C4.2, C5.2, C6.-, C7.-, C8.-, U$1.AGND
- net N$20: now also C2.2, R7.1, R8.1, U1C.-IN; no longer R22.1, VR1.A, VR1.S
- net N$21: now also C2.1, R10.1, U1C.OUT; no longer C23.2, R17.2, R18.1, R6.2
- net N$23: now also C5.2, R21.1, R22.1, U2C.-IN; no longer C27.1, C27.2, C30.+, R19.1, R25.1, U2A.+IN, U2A.OUT
- net N$25: now also OUT1-2.TIP, R10.2, R7.2; no longer D1.A, R5.2
- net N$26: now also OUT2-2.TIP, R21.2, R24.2; no longer C28.2, R20.2, R24.1, R26.2
- net N$28: now also R26.2, TR6.2, TR6.2-2; no longer C29.+, R26.1
- net N$31: now also OUT2-3.TIP, R27.2; no longer C26.2, R19.2, R21.1
- net N$4: now also C4.2, R15.1, R16.1, U2A.-IN; no longer C4.1, C7.+, U$1.FILT+_ADC
- net N$5: now also R18.1, TR4.1; no longer C3.1, C6.+, U$1.FILT+_DAC
- net N$6: now also R3.1, TR1.1; no longer C24.1, R7.1, U1A.OUT
- net N$7: now also C1.1, R2.2, TR1.3, TR2.3, TR3.3, U1A.OUT; no longer R17.1, R23.1, U1C.OUT
- net N$8: now also R19.2, TR4.2, TR4.2-2; no longer C12.+, D4.A, IC1.OUT
- net N$9: now also R4.2, TR1.2, TR1.2-2; no longer C24.2, R11.1, U1A.-IN
- net PWR+12V: now also C25.1, C8.1, U1P.V+, U2P.V+; no longer C11.+, IC1.IN, R15.1
- net PWR-12V: now also C11.2, C7.2, U1P.V-, U2P.V-
Other:
- note removed: "9V Battery & Power Jack"
- note removed: "As drawn: SW1 up = Bypassed SW1 down = Active"
- note removed: "C1 is input coupling cap C2 is output coupling cap. Different circuits will use different values. PCB has dual footprint that accepts 2mm and 5mm radial caps."
- note removed: "Clear SJ1 to disable onboard LED (D1)"
- note removed: "Eurorack input"
- note removed: "FX Goes Here"
- note removed: "Guitar input"
- note removed: "Input, Output and Bypass Circuitry"
- note removed: "LED Active/Bypass indicator"
- note removed: "Near midpoint"
- note removed: "Near power jack"
- note removed: "Nominal Power is 9V battery or 9V wall wart. Wall wart follows the Roland/Boss convention: *Tip is ground. *Sleeve is +9V. Plugging in to the barrel jack takes the battery out of circuit by lifting the sleeve normal. Q1 is wired as ideal diode, to only conduct when power is properly polarized. Reverse polarity isn't conducted, preventing damage if wrong wart is used, or if battery is mistakenly r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"
- note removed: "Power Pins"
- note removed: "Select R2 for brightness of D2"
- note removed: "VAUX is optional auxillary voltage intended for 3.3V or 5V for digital circuits, or buffered VCC/2 reference voltage."
- moved on the sheet: C10, C23, C24, C25, C3, C4, C5, C9, D2, D3, R1, R10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
