File: eagle/euro buffered mult/buffered mult panel.brd (EAGLE design)
At the start: 25.4 x 128.5 mm, 3 parts

Commit message: xr-vco-panel.zip added
Parts:
- added U$1, U$5, U$6, U$7, U$8: (no value), MusicThingModular:TRIMMERHOLE
Other:
- board text added: "Buffered Mult"
- board text added: "Buffered Mult Designed by Zack Hagan Feb 2018 zhagan@gmail.com"
- board text added: "Input"
- board text added: "Out"
- board text removed: "1V/O"
- board text removed: "Dual XR-VCO"
- board text removed: "Exp_FM"
- board text removed: "Sync"
- board text removed: "Thomas Henry XR-VCO PCB design by Zack Hagan zhagan@gmail.com April 2017"
Changed lines of the file:
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@@
 <wire x1="25.4" y1="128.5" x2="0" y2="128.5" width="0" layer="20"/>
 <circle x="9.2" y="31" radius="3.5" width="0.4064" layer="21"/>
-<text x="47" y="115" size="5.08" layer="29" rot="SR0" align="center">Dual XR-VCO</text>
-<text x="45.1193" y="113.531" size="1.4224" layer="26" rot="SMR0" align="center">Thomas Henry XR-VCO
-PCB design by Zack Hagan
-zhagan@gmail.com
-April 2017</text>
+<text x="12" y="118" size="2.54" layer="30" rot="SMR0" align="center">Buffered
+Mult</text>
 <wire x1="0" y1="128.5" x2="0.0175" y2="0.035" width="0" layer="21"/>
-<rectangle x1="0" y1="0" x2="25.4" y2="9" layer="30"/>
-<rectangle x1="-0.1425" y1="119.365" x2="25.4" y2="128.365" layer="30"/>
+<rectangle x1="0" y1="0" x2="25.4" y2="9" layer="29"/>
+<rectangle x1="-0.1425" y1="119.365" x2="25.4" y2="128.365" layer="29"/>
 <circle x="9.2" y="69" radius="3.5" width="0.4064" layer="22"/>
 <circle x="9.2" y="80" radius="3.5" width="0.4064" layer="22"/>
 <circle x="9.2" y="91" radius="3.5" width="0.4064" layer="22"/>
-<text x="73.3407" y="73.941" size="1.778" layer="25" rot="SR0" align="center">Exp_FM</text>
-<text x="85.5487" y="88.591" size="1.778" layer="25" rot="SR0" align="center">1V/O</text>
-<text x="73.6757" y="89.0622" size="1.778" layer="25" rot="SR0" align="center">Sync</text>
+<text x="18.3407" y="101.941" size="1.778" layer="26" rot="SMR0" align="center">Input</text>
+<text x="15.5487" y="47.591" size="1.778" layer="26" rot="SMR0" align="center">Out</text>
+<text x="17.6757" y="54.0622" size="1.778" layer="26" rot="SMR0" align="center">Input</text>
+<text x="13.0232" y="112.941" size="1.6764" layer="25" rot="SR0" align="center">Buffered Mult
+Designed by
+Zack Hagan
+Feb 2018
+zhagan@gmail.com</text>
+<text x="16.5487" y="95.591" size="1.778" layer="26" rot="SMR0" align="center">Out</text>
 </plain>
 <attributes>
@@
 <element name="U$4" library="MusicThingModular" package="SLOT_HOLE" value="" x="7.5175" y="3.035"/>
 <element name="U$2" library="MusicThingModular" package="TRIMMERHOLE" value="" x="17" y="20"/>
+<element name="U$1" library="MusicThingModular" package="TRIMMERHOLE" value="" x="17" y="31"/>
+<element name="U$5" library="MusicThingModular" package="TRIMMERHOLE" value="" x="17" y="42"/>
+<element name="U$6" library="MusicThingModular" package="TRIMMERHOLE" value="" x="17" y="69"/>
+<element name="U$7" library="MusicThingModular" package="TRIMMERHOLE" value="" x="17" y="80"/>
+<element name="U$8" library="MusicThingModular" package="TRIMMERHOLE" value="" x="17" y="91"/>
 </elements>
 <signals>
 <signal name="GND">
 <polygon width="0.4064" layer="16">
-<vertex x="28.5625" y="131.305"/>
+<vertex x="30.5625" y="131.305"/>
 <vertex x="29.1025" y="-3.95"/>
 <vertex x="-2.8575" y="-4.95"/>
-<vertex x="-5.3975" y="130.305"/>
+<vertex x="-3.3975" y="130.305"/>
 </polygon>
 <via x="9.2" y="20" extent="1-16" drill="6"/>
