File: eagle/teensy_pedal/Proto_Pedal/teensy_pedal.sch (EAGLE design)
At the start: 29 parts, among them Q1 2.5A/30V, U1 TL074_SMD, U2 TL074_SMD

Commit message: add euro buffer
Parts:
- added C10, C12, C17, C22, C9: 10uf, resistor:CPOL-US153CLV-0505
- added C11, C29, C30, C35, C36, C7: 22uf, resistor:CPOL-US153CLV-0605
- added C13, C14, C18, C19, C3, C5: 0.1uf, resistor:C-USC0603
- added C15, C16, C20, C21: 0.01uf, resistor:C-USC0603
- added C23, C40, C43, C46: 4.7uf 0805, resistor:C-USC0805
- added C24, C38, C41, C44: 470pf, resistor:C-USC0603
- added C25, C27, C33, C39, C42, C45: 2700pf, resistor:C-USC0603
- added C26, C32: 1800pf, resistor:C-USC0603
- added C28, C34: 5600pf, resistor:C-USC0603
- added C31, C37: 1200pf, resistor:C-USC0603
- added C4: o.1uf, resistor:C-USC0603
- added C6: 100uf, resistor:CPOL-US153CLV-0810
- added C8: 4.7uf, resistor:CPOL-US153CLV-0505
- added D2, D3, D4: 1N4004, diode:1N4004
- added IC1: 7805, v-reg:78XXS
- added R10, R13, R14, R15, R23, R41, R43, R44, R46, R47, R49, R50, R52, R53, R55, R56, R58, R59, R6, R8: 100k, resistor:R-US_R0603
- added R11, R45, R51, R57: 634, resistor:R-US_R0603
- added R12: 150R, resistor:R-US_R0603
- added R16: 20k, resistor:R-US_R0603
- added R17, R18: 1k, resistor:R-US_R0603
- added R19, R29: 2.94k, resistor:R-US_R0603
- added R20, R30: 887R, resistor:R-US_R0603
- added R21, R31: 5.49k, resistor:R-US_R0603
- added R22: 1M, resistor:R-US_R0603
- added R24, R32: 1.65k, resistor:R-US_R0603
- added R25, R33: 4.75k, resistor:R-US_R0603
- added R26, R34: 1.87k, resistor:R-US_R0603
- added R27, R35: 562R, resistor:R-US_R0603
- added R28, R36: 47.5k, resistor:R-US_R0603
- added R37, R38: 24k, resistor:R-US_R0603
- added R39: 220R, resistor:R-US_R0603
- added R40: 220, resistor:R-US_R0603
- added R42, R48, R54, R7: 91, resistor:R-US_R0603
- added R9: 27k, resistor:R-US_R0603
- added SV1: EURO_POWER_HEADERFAT_PADS, MusicThingModular:EURO_POWER_HEADERFAT_PADS
- added U$3: CAT811, sot143:CAT811
- added U3, U4, U5: TL072_SMD, MusicThingModular:TL072_SMD
- added VR1: 1M, MusicThingModular:9MM_SNAP-IN_POT_
- added VR2, VR3: b100k, MusicThingModular:9MM_SNAP-IN_POT_
- U1: value TL074_SMD -> TL072_SMD; device MusicThingModular:TL074_SMD -> MusicThingModular:TL072_SMD
Connections:
- new net BCLK: U$1.ADC_SCLK, U$1.DAC_SCLK, U$2.9/CS
- new net LRCLK: U$1.ADC_LRCK, U$1.DAC_LRCK, U$2.23/A9
- new net MCLK: U$1.MCLK, U$2.11/MOSI
- new net N$1: R12.2, R13.2, U$1.CS
- new net N$10: C23.1, R10.2, R8.1, U1A.+IN
- new net N$11: R37.1, U2D.-IN, VR3.A, VR3.S
- new net N$12: R15.2, R16.1
- new net N$13: R18.2, R9.1
- new net N$14: R14.2, R9.2
- new net N$15: R14.1
- new net N$16: C30.-, R27.2
- new net N$17: R27.1, R28.1, U2C.+IN
- new net N$18: C31.1, R20.1, U2A.+IN
- new net N$19: R22.1, VR1.A, VR1.S
- new net N$2: C3.2, C4.2, C5.2, C6.-, C7.-, C8.-, U$1.AGND
- new net N$20: C23.2, R23.1, U1B.OUT
- new net N$21: R18.1, R6.2
- new net N$22: R22.2
- new net N$23: C27.1, C27.2, C30.+, R19.1, R25.1, U2A.-IN, U2A.OUT
- new net N$24: R38.1, U2C.-IN, VR2.A, VR2.S
- new net N$26: C28.2, R20.2, R24.1, R26.2
- new net N$27: R40.2, U2D.OUT, VR3.E
- new net N$28: C29.+, R26.1
- new net N$29: R39.2, U2C.OUT, VR2.E
- new net N$30: R39.1
- new net N$31: C26.2, R19.2, R21.1, R25.2
- new net N$32: C36.-, R35.2
- new net N$33: R35.1, R36.1, U2D.+IN
- new net N$34: C37.1, R30.1, U2B.+IN
- new net N$36: C33.1, C33.2, C36.+, R29.1, R33.1, U2B.-IN, U2B.OUT
- new net N$37: C34.2, R30.2, R32.1, R34.2
- new net N$38: C35.+, R34.1
- new net N$39: C32.2, R29.2, R31.1, R33.2
- new net N$4: C4.1, C7.+, U$1.FILT+_ADC
- new net N$40: R40.1
- new net N$41: R23.2, R41.1, U1B.-IN
- new net N$42: C38.1, R42.1, U3A.OUT
- new net N$43: C38.2, R45.1, U3A.-IN
- new net N$44: C40.1, R43.1, R44.2, U3A.+IN
- new net N$46: C40.2, R46.1, U3B.OUT
- new net N$47: R46.2, R47.1, U3B.-IN
- new net N$48: C41.1, R48.1, U4A.OUT
- new net N$49: C41.2, R51.1, U4A.-IN
- new net N$5: C3.1, C6.+, U$1.FILT+_DAC
- new net N$50: C43.1, R49.1, R50.2, U4A.+IN
- new net N$51: C43.2, R52.1, U4B.OUT
- new net N$52: R52.2, R53.1, U4B.-IN
- new net N$53: C44.1, R54.1, U5A.OUT
- new net N$54: C44.2, R57.1, U5A.-IN
- new net N$56: C46.1, R55.1, R56.2, U5A.+IN
- new net N$57: C46.2, R58.1, U5B.OUT
- new net N$58: R58.2, R59.1, U5B.-IN
- new net N$6: C24.1, R7.1, U1A.OUT
- new net N$7: R17.1, VR1.E
- new net N$8: C12.+, D4.A, IC1.OUT
- new net N$9: C24.2, R11.1, U1A.-IN
- new net PWR+12V: C11.+, C9.+, D2.C, IC1.IN, R15.1, SV1.10, SV1.9
- new net PWR-12V: C10.-, D3.A, SV1.1, SV1.2
- new net PWR33V: C13.1, C14.1, C15.1, C16.1, C17.+, R13.1, U$1.VD, U$1.VD1, U$1.VLC, U$1.VLS, U$2.3V3
- new net PWR5V: C18.1, C19.1, C20.1, C21.1, C22.+, D4.C, R43.2, R49.2, R55.2, R8.2, U$1.VA, U$1.VA1, U$2.VIN
- new net RESET: U$1.RST
- new net RX: U$1.ADC_SDOUT1, U$2.13/SCK
- new net SCL: U$1.SCL/CCLK, U$2.19/A5/SCL
- new net SDA: U$1.SDA/CDOUT, U$2.18/A4/SDA
- new net TOAIN1: C25.1, C42.1, R11.2, R48.2, R51.2, R7.2
- new net TOAIN2: C39.1, R42.2, R45.2
- new net TOAIN3: C45.1, R54.2, R57.2
- new net TX: U$1.DAC_SDIN1, U$2.22/A8
- new net VQ: C5.1, C8.+, U$1.VQ
- net GND: now also C10.+, C11.-, C12.-, C13.2, C14.2, C15.2, C16.2, C17.-, C18.2, C19.2, C20.2, C21.2, C22.-, C25.2, C26.1, C28.1, C29.-, C31.2, C32.1, C34.1, C35.-, C37.2, C39.2, C42.2, C45.2, C9.-, D2.A, D3.C, IC1.GND, R10.1, R12.1, R16.2, R28.2, R36.2, R37.2, R38.2, R44.1, R50.1, R56.1, R6.1, SV1.3, SV1.4, SV1.5, SV1.6, SV1.7, SV1.8, U$1.AUX_SCLK, U$1.AUX_SDIN, U$1.CDIN, U$1.DAC_SDIN2, U$1.DAC_SDIN3, U$1.DAC_SDIN4, U1B.+IN, U3B.+IN, U4B.+IN, U5B.+IN
Other:
- note added: "Eurorack input"
- note added: "Guitar input"
- moved on the sheet: U1A, U1B, U2A, U2B, U2C, U2D
